File: SchematicDiagram/rocket.kicad_sch (KiCad schematic)
At the start: 12 parts, among them IC1 NJM2819ADL3-33-TE1, SW1 SW_Push, SW2 SW_Push, U1 ESP32-DevKitC

Commit message: NJM2396F33
Parts:
- removed C1, C2: 4.7μC, symbol Device:C
- removed IC1: NJM2819ADL3-33-TE1, NJM2819ADL333TE1, symbol NJM2819ADL3-33-TE1:NJM2819ADL3-33-TE1
- removed R2: 10kΩ, symbol Device:R
- removed SW2: SW_Push, symbol Switch:SW_Push
- added C3: 0.33μC, symbol Device:C
- added C4: 22μC, symbol Device:C
- added SW3: SW_Push, symbol Switch:SW_Push
- added U2: NJM2396F33, TO254P480X1000X1900-4P, symbol NJM2396F33:NJM2396F33
Connections:
- net 3.3V: now also C4.2, U2.2 (VOUT)
- net GND: now also C3.2, C4.1, U2.3 (GND)
- net VCC: now also SW3.2
- new net: C3.1, SW3.1, U2.1 (VIN), U2.4 (ON/OFF_CONTROL)
- no-connect marks 10 -> 8
